File: hardware/nucleum/rev_a/nucleum.brd (EAGLE design)
At the start: 18.8 x 19.6 mm, 40 parts, among them J1 TC2030-JLINK-NL, J2 SH_MALE_2/1MM, J3 ATUM-HEADER, U2 FM25LBTDFN-8, U3 RV-3049-C3, U4 TPS62740, U5 NRF51822QF, X1 EPSON-FA-128, X2 ABS05-32.768KHZ-T

Commit message: finished layout and routing
Parts:
- moved J1 0.73 mm to (3.26, 9.65)
- moved R3 0.15 mm to (8.19, 10.8)
- moved R9 0.06 mm to (1.36, 15.1)
- moved R10 0.06 mm to (0.50, 15.1)
Routing:
- net SWDIO/!RESET: track 28.0 -> 31.1 mm
- net SWDCLK: track 29.1 -> 28.0 mm
- net LED_GREEN: track 12.6 -> 13.6 mm, vias 0 -> 2
- net P17: track 19.8 -> 19.0 mm
- net VCC: track 14.5 -> 13.8 mm
- net GND: track 22.0 -> 21.9 mm, vias 49 -> 28
Other:
- board text added: "Joshua Adkins"
- board text added: "Rev_A"
- board text removed: "Joshua Adkins Brad Campbell"

Commit message: regain board annotation, finished/fix annotation erros
Parts:
- removed C17: 1nF, passives:0402_CAP
- removed C18: 47nF, passives:0402_CAP
- removed C21: 2.2nF, passives:0402_CAP
- removed C22: 0.8pF, passives:0402_CAP
- removed R10, R8, R9: 1k, passives:0402_RES
- removed U2: FM25LBTDFN-8, chips:TDFN-8
- added C12: 0.1uF, passives:0402_CAP
- added C13: 1uF, passives:0402_CAP
- added C14: 4.7uF, passives:0402_CAP
- added C6: 1nF, passives:0402_CAP
- added R4, R5: 10k, passives:0402_RES
- added R6: 12k, passives:0402_RES
- added U1: FM25L04B-DG, chips:TDFN-8
- C1: value 12pF -> 0.8pF
- C10: value 4.7uF -> 47nF
- C11: value 1uF -> 0.1uF
- C3, C4: value 22pF -> 12pF
- C5: value 1nF -> 12pF
- C7: value 10nF -> 1nF
- C8: value 0.1uF -> 2.2nF
- C9: value 0.1uF -> 10nF
- L1: value 2.2 -> 15nH; device passives:MIPSZ201D -> passives:0402_CAP
- L2: value (none) -> 2.2uH; device passives:0402_CAP -> passives:MIPSZ201D
- L3: value (none) -> 10uH
- R1, R2: value 10k -> 1k
- R3: value 12k -> 1k
- moved C7 16.1 mm to (10.2, 1.58), turned to 270 degrees
- moved R1 15.2 mm to (1.36, 15.1), turned to 90 degrees
- moved R2 14.6 mm to (0.50, 15.1), turned to 90 degrees
- moved C8 12.7 mm to (4.65, 7.67), turned to 90 degrees
- moved L1 12.0 mm to (5.52, 4.66), flipped to the top
- moved L2 12.0 mm to (1.93, 16.1), flipped to the bottom
- moved C11 10.5 mm to (16.8, 4.33), turned to 270 degrees
- moved C3 10.4 mm to (6.02, 0.68)
- moved C5 9.97 mm to (16.4, 1.27), turned to 0 degrees
- moved C10 9.52 mm to (5.91, 7.62)
- moved R3 7.42 mm to (2.17, 15.1), turned to 90 degrees
- moved C1 7.31 mm to (3.84, 7.66), turned to 90 degrees
- moved C9 5.30 mm to (14.5, 17.1), turned to 180 degrees
- renumbered C19 to C15, C20 to C16, U$1 to S1
Connections:
- removed net N$1: J3.30, J3.30B
- new net UNUSED1: J3.5, J3.5B
- new net UNUSED2: J3.10, J3.10B
- new net UNUSED3: J3.11, J3.11B
- new net UNUSED4: J3.12, J3.12B
- new net UNUSED5: J3.13, J3.13B
- net !FRAM_CS: now also U1.1; no longer U2.1
- net !FRAM_HOLD: now also U1.7; no longer U2.7
- net !FRAM_WP: now also U1.3; no longer U2.3
- net ANTENNA: now also C1.1; no longer C22.1
- net GND: now also C12.2, C13.2, C14.2, C6.2, R4.2, R5.2, R6.1, U1.4, U5.13, U5.33, U5.34, U5.GND; no longer C17.2, C18.2, C21.2, C22.2, R1.2, R2.2, R3.1, U2.4
- net LED_BLUE: now also R1.1; no longer R9.1
- net LED_GREEN: now also R2.1; no longer R10.1
- net LED_RED: now also R3.1; no longer R8.1
- net N$11: now also R2.2; no longer R10.2
- net N$12: now also R1.2; no longer R9.2
- net N$14: now also R4.1; no longer R2.1
- net N$15: now also C10.1; no longer C18.1
- net N$16: now also R5.1; no longer R1.1
- net N$17: now also C7.1; no longer C17.1
- net N$20: now also C8.1; no longer C21.1
- net N$36: now also C13.1, C6.1, L1.1; no longer C11.1, C5.1, L2.1
- net N$37: now also L1.2; no longer L2.2
- net N$5: now also L2.1; no longer L1.1
- net N$6: now also C5.1; no longer C3.1
- net N$7: now also R3.2; no longer R8.2
- net N$9: now also C3.1; no longer C1.1
- net SPI_MISO: now also U1.2; no longer U2.2
- net SPI_MOSI: now also U1.5; no longer U2.5
- net SPI_SCK: now also U1.6; no longer U2.6
- net SWDCLK: now also R6.2; no longer R3.2
- net SWDIO/!RESET: now also J3.3, J3.30, J3.30B, J3.3B; no longer J3.5, J3.5B
- net VCC: now also C11.1, C12.1, C14.1, L2.2, U1.8; no longer C10.1, C7.1, C8.1, L1.2, U2.8
Routing:
- net SWDIO/!RESET: track 31.1 -> 37.8 mm, vias 2 -> 3
- net GND: track 21.9 -> 23.2 mm
