File: hardware/nucleum/rev_a/nucleum.sch (EAGLE design)
At the start: 40 parts, among them J1 TC2030-JLINK-NL, J2 SH_MALE_2/1MM, J3 ATUM-HEADER, U2 FM25LBTDFN-8, U3 RV-3049-C3, U4 TPS62740, U5 NRF51822QF, X1 EPSON-FA-128, X2 ABS05-32.768KHZ-T

Commit message: regain board annotation, finished/fix annotation erros
Parts:
- removed C17: 1nF, passives:CAPACITOR
- removed C18: 47nF, passives:CAPACITOR
- removed C21: 2.2nF, passives:CAPACITOR
- removed C22: 0.8pF, passives:CAPACITOR
- removed R10, R8, R9: 1k, passives:RESISTOR0402_RES
- removed U2: FM25LBTDFN-8, chips:FM25LBTDFN-8
- added C12: 0.1uF, passives:CAPACITOR
- added C13: 1uF, passives:CAPACITOR
- added C14: 4.7uF, passives:CAPACITOR
- added C6: 1nF, passives:CAPACITOR
- added R4, R5: 10k, passives:RESISTOR0402_RES
- added R6: 12k, passives:RESISTOR0402_RES
- added U1: FM25L04B-DG, chips:FM25L04B-DG
- C1: value 12pF -> 0.8pF
- C10: value 4.7uF -> 47nF
- C11: value 1uF -> 0.1uF
- C3, C4: value 22pF -> 12pF
- C5: value 1nF -> 12pF
- C7: value 10nF -> 1nF
- C8: value 0.1uF -> 2.2nF
- C9: value 0.1uF -> 10nF
- L1: value 2.2 -> 15nH; device passives:MIPSZ2012D -> passives:INDUCTOR0402
- L2: value (none) -> 2.2uH; device passives:INDUCTOR0402 -> passives:MIPSZ2012D
- L3: value (none) -> 10uH
- R1, R2: value 10k -> 1k
- R3: value 12k -> 1k
- renumbered C19 to C15, C20 to C16, U$1 to S1
Connections:
- net !FRAM_CS: now also U1.!CS; no longer U2.!CS
- net !FRAM_HOLD: now also U1.!HOLD; no longer U2.!HOLD
- net !FRAM_WP: now also U1.!WP; no longer U2.!WP
- net ANTENNA: now also C1.1; no longer C22.1
- net GND: now also C12.2, C13.2, C14.2, C6.2, R4.2, R5.2, R6.1, U1.VSS, U5.GND; no longer C17.2, C18.2, C21.2, C22.2, R1.2, R2.2, R3.1, U2.VSS
- net LED_BLUE: now also R1.1; no longer R9.1
- net LED_GREEN: now also R2.1; no longer R10.1
- net LED_RED: now also R3.1; no longer R8.1
- net N$11: now also R2.2; no longer R10.2
- net N$12: now also R1.2; no longer R9.2
- net N$14: now also R4.1; no longer R2.1
- net N$15: now also C10.1; no longer C18.1
- net N$16: now also R5.1; no longer R1.1
- net N$17: now also C7.1; no longer C17.1
- net N$20: now also C8.1; no longer C21.1
- net N$36: now also C13.1, C6.1, L1.1; no longer C11.1, C5.1, L2.1
- net N$37: now also L1.2; no longer L2.2
- net N$5: now also L2.1; no longer L1.1
- net N$6: now also C5.1; no longer C3.1
- net N$7: now also R3.2; no longer R8.2
- net N$9: now also C3.1; no longer C1.1
- net SPI_MISO: now also U1.SO; no longer U2.SO
- net SPI_MOSI: now also U1.SI; no longer U2.SI
- net SPI_SCK: now also U1.SCK; no longer U2.SCK
- net SWDCLK: now also R6.2; no longer R3.2
- net VCC: now also C11.1, C12.1, C14.1, L2.2, U1.VDD; no longer C10.1, C7.1, C8.1, L1.2, U2.VDD
