File: hardware/nucleum_logger/nucleum_logger.brd (EAGLE design)
At the start: 30.5 x 69.9 mm, 7 parts, among them J1 DM3AT-SF-PEJM5, J3 SQUALL_HEADERSQUALL_CARRIER, U1 NUCLEUM

Commit message: did some final changes to the nucleum logger board
Parts:
- renumbered U$1 to J2
Other:
- board text added: "BLEES Compatible Shield"
- board text added: "Nucleum Logger Rev_A Joshua Adkins - Lab11 June 2016"
Changed lines of the file:
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@@
 <wire x1="30.48" y1="69.85" x2="-0.0254" y2="69.8502" width="0" layer="20"/>
 <wire x1="-0.0254" y1="69.8502" x2="0" y2="0" width="0" layer="20"/>
+<text x="7.0104" y="49.0982" size="1.016" layer="25">BLEES Compatible Shield</text>
+<text x="7.0612" y="18.6182" size="1.016" layer="25">Nucleum Logger Rev_A
+Joshua Adkins - Lab11
+June 2016
+</text>
 </plain>
 <attributes>
@@
 </autorouter>
 <elements>
-<element name="J1" library="connector" package="DM3AT-SF-PEJM5" value="DM3AT-SF-PEJM5" x="13.97" y="32.2834" rot="R90">
+<element name="J1" library="connector" package="DM3AT-SF-PEJM5" value="DM3AT-SF-PEJM5" x="13.97" y="32.2834" smashed="yes" rot="R90">
 <attribute name="DIGIKEY" value="HR1964CT-ND" x="52.07" y="56.4134" size="1.778" layer="27" rot="R90" display="off"/>
+<attribute name="NAME" x="14.9546" y="39.9938" size="1.016" layer="25" font="vector" ratio="12" align="bottom-center"/>
 </element>
-<element name="J3" library="squall" package="SQUALL_CARRIER" value="SQUALL_HEADERSQUALL_CARRIER" x="15.24" y="56.5404"/>
+<element name="J3" library="squall" package="SQUALL_CARRIER" value="SQUALL_HEADERSQUALL_CARRIER" x="15.24" y="56.5404" smashed="yes">
+<attribute name="NAME" x="15.2908" y="58.4708" size="1.016" layer="26" font="vector" ratio="12" rot="R180" align="center"/>
+</element>
 <element name="U1" library="nucleum" package="NUCLEUM" value="NUCLEUM" x="16.1036" y="17.9578" rot="R90"/>
-<element name="R2" library="passives" package="0402_RES" value="10K" x="11.3792" y="33.1724" rot="R180"/>
-<element name="R3" library="passives" package="0402_RES" value="10K" x="11.2522" y="35.56" rot="R180"/>
-<element name="U$1" library="connector" package="AA_SMD" value="AA_BAT_PACKSMD" x="15.24" y="34.925" rot="MR0"/>
-<element name="R1" library="passives" package="0402_RES" value="10K" x="25.9842" y="22.0218"/>
+<element name="R2" library="passives" package="0402_RES" value="10K" x="11.3792" y="33.1724" smashed="yes" rot="R180">
+<attribute name="NAME" x="9.779" y="32.7152" size="1.016" layer="25" font="vector" ratio="12" align="bottom-center"/>
+</element>
+<element name="R3" library="passives" package="0402_RES" value="10K" x="11.2522" y="35.56" smashed="yes" rot="R180">
+<attribute name="NAME" x="12.1158" y="37.1602" size="1.016" layer="25" font="vector" ratio="12" rot="R180" align="bottom-center"/>
+</element>
+<element name="J2" library="connector" package="AA_SMD" value="AA_BAT_PACKSMD" x="15.24" y="34.925" rot="MR0"/>
+<element name="R1" library="passives" package="0402_RES" value="10K" x="25.9842" y="22.0218" smashed="yes">
+<attribute name="NAME" x="26.3906" y="22.5044" size="1.016" layer="25" font="vector" ratio="12" align="bottom-center"/>
+</element>
 </elements>
 <signals>
@@
 <vertex x="30.48" y="0.0254"/>
 </polygon>
-<contactref element="U$1" pad="1-"/>
+<contactref element="J2" pad="1-"/>
 <wire x1="7.0247" y1="8.4789" x2="15.6417" y2="8.4789" width="0.508" layer="1"/>
 <wire x1="15.6417" y1="8.4789" x2="15.6718" y2="8.509" width="0.508" layer="1"/>
@@
 <contactref element="R3" pad="2"/>
 <contactref element="R2" pad="2"/>
-<contactref element="U$1" pad="2+"/>
+<contactref element="J2" pad="2+"/>
 <contactref element="R1" pad="2"/>
 <wire x1="4.395" y1="59.8804" x2="3.6702" y2="59.8804" width="0.2032" layer="1"/>
@@
 </signal>
 <signal name="N$1">
-<contactref element="U$1" pad="1+"/>
-<contactref element="U$1" pad="2-"/>
+<contactref element="J2" pad="1+"/>
+<contactref element="J2" pad="2-"/>
 <wire x1="8.128" y1="65.659" x2="22.352" y2="65.659" width="1.27" layer="16"/>
 </signal>
@@
 </board>
 </drawing>
+<compatibility>
+<note version="6.3" minversion="6.2.2" severity="warning">
+Since Version 6.2.2 text objects can contain more than one line,
+which will not be processed correctly with this version.
+</note>
+</compatibility>
 </eagle>
