File: hardware/nucleum_logger/nucleum_logger.sch (EAGLE design)
At the start: 7 parts, among them J1 DM3AT-SF-PEJM5, J3 SQUALL_HEADERSQUALL_CARRIER, U1 NUCLEUM

Commit message: did some final changes to the nucleum logger board
Parts:
- removed U$1: AA_BAT_PACKSMD, connector:AA_BAT_PACKSMD
- added J2: AA_BAT_PACKSMD, connector:AA_BAT_PACKSMD
Connections:
- net GND: now also J2.P1-; no longer U$1.P1-
- net N$1: now also J2.P1+, J2.P2-; no longer U$1.P1+, U$1.P2-
- net VCC: now also J2.P2+; no longer U$1.P2+
Other:
- note removed: "NUCLEUM AIN and DIO PINS are not multiplexed to each squall header. This prevents hardware conflicts between the headers."
- note removed: "SQUALL_HEADER #2"
Changed lines of the file:
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@@
 <part name="R2" library="passives" deviceset="RESISTOR" device="0402_RES" value="10K"/>
 <part name="R3" library="passives" deviceset="RESISTOR" device="0402_RES" value="10K"/>
-<part name="U$1" library="connector" deviceset="AA_BAT_PACK" device="SMD"/>
+<part name="J2" library="connector" deviceset="AA_BAT_PACK" device="SMD"/>
 <part name="R1" library="passives" deviceset="RESISTOR" device="0402_RES" value="10K"/>
 </parts>
@@
 <wire x1="91.44" y1="48.26" x2="91.44" y2="0" width="0.1524" layer="97"/>
 <text x="15.24" y="48.26" size="1.778" layer="97">Micro SD Card Connector</text>
-<text x="2.54" y="175.26" size="1.778" layer="97">NUCLEUM
-AIN and DIO PINS are not multiplexed to each squall header.
-This prevents hardware conflicts between the headers.</text>
 <wire x1="167.64" y1="35.56" x2="167.64" y2="114.3" width="0.1524" layer="97"/>
-<wire x1="167.64" y1="114.3" x2="248.92" y2="114.3" width="0.1524" layer="97"/>
 <wire x1="167.64" y1="114.3" x2="167.64" y2="185.42" width="0.1524" layer="97"/>
 <text x="193.04" y="180.34" size="1.778" layer="97">SQUALL HEADER #1</text>
-<text x="193.04" y="109.22" size="1.778" layer="97">SQUALL_HEADER #2</text>
-<text x="119.38" y="124.46" size="1.778" layer="97">BATTERY</text>
-<text x="119.38" y="86.36" size="1.778" layer="97">TWO AA's</text>
+<text x="121.92" y="116.84" size="1.778" layer="97">BATTERY</text>
+<text x="121.92" y="93.98" size="1.778" layer="97">TWO AA's</text>
 </plain>
 <instances>
@@
 <instance part="GND5" gate="1" x="50.8" y="17.78"/>
 <instance part="GND6" gate="1" x="35.56" y="5.08"/>
-<instance part="GND7" gate="1" x="134.62" y="106.68"/>
+<instance part="GND7" gate="1" x="106.68" y="116.84"/>
 <instance part="J3" gate="G$1" x="205.74" y="152.4"/>
 <instance part="U1" gate="G$1" x="45.72" y="119.38"/>
@@
 <instance part="R2" gate="G$1" x="63.5" y="33.02" rot="R90"/>
 <instance part="R3" gate="G$1" x="48.26" y="33.02" rot="R90"/>
-<instance part="U$1" gate="G$1" x="99.06" y="109.22"/>
+<instance part="J2" gate="G$1" x="116.84" y="106.68"/>
 <instance part="R1" gate="G$1" x="78.74" y="30.48" rot="R90"/>
 </instances>
@@
 </segment>
 <segment>
-<wire x1="127" y1="111.76" x2="127" y2="114.3" width="0.1524" layer="91"/>
-<wire x1="127" y1="114.3" x2="134.62" y2="114.3" width="0.1524" layer="91"/>
-<wire x1="134.62" y1="114.3" x2="134.62" y2="109.22" width="0.1524" layer="91"/>
+<wire x1="106.68" y1="121.92" x2="106.68" y2="119.38" width="0.1524" layer="91"/>
 <pinref part="GND7" gate="1" pin="GND"/>
-<wire x1="127" y1="114.3" x2="127" y2="137.16" width="0.1524" layer="91"/>
-<junction x="127" y="114.3"/>
-<pinref part="U$1" gate="G$1" pin="P1-"/>
-<wire x1="127" y1="137.16" x2="93.98" y2="137.16" width="0.1524" layer="91"/>
-<wire x1="93.98" y1="137.16" x2="93.98" y2="121.92" width="0.1524" layer="91"/>
+<pinref part="J2" gate="G$1" pin="P1-"/>
+<wire x1="106.68" y1="121.92" x2="114.3" y2="121.92" width="0.1524" layer="91"/>
+<wire x1="114.3" y1="121.92" x2="114.3" y2="119.38" width="0.1524" layer="91"/>
 </segment>
 <segment>
@@
 </segment>
 <segment>
-<label x="121.92" y="114.3" size="1.27" layer="95" rot="R90" xref="yes"/>
-<wire x1="121.92" y1="114.3" x2="121.92" y2="109.22" width="0.1524" layer="91"/>
-<wire x1="121.92" y1="109.22" x2="114.3" y2="109.22" width="0.1524" layer="91"/>
-<wire x1="114.3" y1="109.22" x2="114.3" y2="127" width="0.1524" layer="91"/>
-<pinref part="U$1" gate="G$1" pin="P2+"/>
-<wire x1="114.3" y1="127" x2="106.68" y2="127" width="0.1524" layer="91"/>
-<wire x1="106.68" y1="127" x2="106.68" y2="121.92" width="0.1524" layer="91"/>
+<label x="119.38" y="129.54" size="1.27" layer="95" rot="R90" xref="yes"/>
+<pinref part="J2" gate="G$1" pin="P2+"/>
+<wire x1="119.38" y1="129.54" x2="119.38" y2="119.38" width="0.1524" layer="91"/>
 </segment>
 <segment>
@@
 <net name="N$1" class="0">
 <segment>
-<pinref part="U$1" gate="G$1" pin="P1+"/>
-<wire x1="93.98" y1="86.36" x2="93.98" y2="81.28" width="0.1524" layer="91"/>
-<pinref part="U$1" gate="G$1" pin="P2-"/>
-<wire x1="93.98" y1="81.28" x2="106.68" y2="81.28" width="0.1524" layer="91"/>
-<wire x1="106.68" y1="81.28" x2="106.68" y2="86.36" width="0.1524" layer="91"/>
+<pinref part="J2" gate="G$1" pin="P1+"/>
+<wire x1="114.3" y1="93.98" x2="114.3" y2="91.44" width="0.1524" layer="91"/>
+<pinref part="J2" gate="G$1" pin="P2-"/>
+<wire x1="114.3" y1="91.44" x2="119.38" y2="91.44" width="0.1524" layer="91"/>
+<wire x1="119.38" y1="91.44" x2="119.38" y2="93.98" width="0.1524" layer="91"/>
 </segment>
 </net>
@@
 </schematic>
 </drawing>
-<compatibility>
-<note version="6.3" minversion="6.2.2" severity="warning">
-Since Version 6.2.2 text objects can contain more than one line,
-which will not be processed correctly with this version.
-</note>
-</compatibility>
 </eagle>
